Commit message: added periodic joints as a setable config. need to figure out how to handle normalizing all other joints (vel with inf as space)... also need to update config for all other models which will be easy.

File: gym_bb/models/models/monopod-fixed/monopod-fixed.urdf (robot description, URDF)
Before this commit: robot monopod-fixed, 6 links, 5 joints
Joints:
- joint knee_joint: limit lower=-6.28 upper=6.28 effort=50 velocity=3.1415926535916 -> (none); type revolute -> continuous

File: gym_bb/models/models/monopod-fixed_hip/monopod-fixed_hip.urdf (robot description, URDF)
Before this commit: robot monopod-fixed_hip, 6 links, 5 joints
Joints:
- joint knee_joint: limit lower=-6.28 upper=6.28 effort=50 velocity=3.1415926535916 -> (none); type revolute -> continuous

File: gym_bb/models/models/monopod-old-fixed/monopod-old-fixed.urdf (robot description, URDF)
Before this commit: robot monopod-old-fixed, 7 links, 6 joints
Joints:
- joint knee_joint: limit lower=-6.28 upper=6.28 effort=50 velocity=3.1416 -> (none); type revolute -> continuous

File: gym_bb/models/models/monopod-old-fixed_hip/monopod-old-fixed_hip.urdf (robot description, URDF)
Before this commit: robot monopod-old-fixed_hip, 7 links, 6 joints
Joints:
- joint knee_joint: limit lower=-6.28 upper=6.28 effort=50 velocity=3.1416 -> (none); type revolute -> continuous

File: gym_bb/models/models/monopod-old/monopod-old.urdf (robot description, URDF)
Before this commit: robot monopod-old, 7 links, 6 joints
Joints:
- joint knee_joint: limit lower=-6.28 upper=6.28 effort=50 velocity=3.1416 -> (none); type revolute -> continuous

File: gym_bb/models/models/monopod/monopod.urdf (robot description, URDF)
Before this commit: robot monopod, 6 links, 5 joints
Joints:
- joint knee_joint: limit lower=-6.28 upper=6.28 effort=50 velocity=3.1415926535916 -> (none); type revolute -> continuous
