Commit message: Made knee joints continuous

File: gym_os2r/models/models/monopod-fixed/monopod-fixed.urdf (robot description, URDF)
Before this commit: robot monopod-fixed, 6 links, 5 joints
Joints:
- joint hip_joint: limit lower=-6.28 upper=6.28 effort=50 velocity=3.1415926535916 -> (none); type revolute -> continuous

File: gym_os2r/models/models/monopod-fixed_hip/monopod-fixed_hip.urdf (robot description, URDF)
Before this commit: robot monopod-fixed_hip, 6 links, 5 joints
Joints:
- joint hip_joint: limit lower=-6.28 upper=6.28 effort=50 velocity=3.1415926535916 -> (none); type revolute -> continous

File: gym_os2r/models/models/monopod/monopod.urdf (robot description, URDF)
Before this commit: robot monopod, 6 links, 5 joints
Joints:
- joint hip_joint: limit lower=-6.28 upper=6.28 effort=50 velocity=3.1415926535916 -> (none); type revolute -> continuous

Commit message: fixed the randomizer. Now randomizes model and world surface.

File: gym_os2r/models/models/monopod-fixed/monopod-fixed.urdf (robot description, URDF)
Before this commit: robot monopod-fixed, 6 links, 5 joints
Links:
- link central_pivot_link: geometry collision mesh filename=package://monopod-fixed/meshes/central_pivot.STL; visual mesh filename=package://monopod-fixed/meshes/central_pivot.STL

File: gym_os2r/models/models/monopod-fixed_hip/monopod-fixed_hip.urdf (robot description, URDF)
Before this commit: robot monopod-fixed_hip, 6 links, 5 joints
Links:
- link central_pivot_link: geometry collision mesh filename=package://monopod-fixed_hip/meshes/central_pivot.STL; visual mesh filename=package://monopod-fixed_hip/meshes/central_pivot.STL

File: gym_os2r/models/models/monopod-simple/monopod-simple.urdf (robot description, URDF)
Before this commit: robot monopod-simple, 6 links, 5 joints
Links:
- link central_pivot_link: geometry collision mesh filename=package://monopod-simple/meshes/central_pivot.STL; visual mesh filename=package://monopod-simple/meshes/central_pivot.STL

File: gym_os2r/models/models/monopod/monopod.urdf (robot description, URDF)
Before this commit: robot monopod, 6 links, 5 joints
Links:
- link central_pivot_link: geometry collision mesh filename=package://monopod/meshes/central_pivot.STL; visual mesh filename=package://monopod/meshes/central_pivot.STL

Commit message: fixed masses

File: gym_os2r/models/models/monopod-fixed/monopod-fixed.urdf (robot description, URDF)
Before this commit: robot monopod-fixed, 6 links, 5 joints
Links:
- link boom_link: mass 0.12458 -> 0.692

File: gym_os2r/models/models/monopod-fixed_hip/monopod-fixed_hip.urdf (robot description, URDF)
Before this commit: robot monopod-fixed_hip, 6 links, 5 joints
Links:
- link boom_link: mass 0.12458 -> 0.692

File: gym_os2r/models/models/monopod-simple/monopod-simple.urdf (robot description, URDF)
Before this commit: robot monopod-simple, 6 links, 5 joints
Links:
- link boom_link: mass 0.12458 -> 0.692

File: gym_os2r/models/models/monopod/monopod.urdf (robot description, URDF)
Before this commit: robot monopod, 6 links, 5 joints
Links:
- link boom_link: mass 0.414 -> 0.692
